File: better-klipper-expander.kicad_pcb (KiCad board)
At the start: 4 copper layers, 105 x 32 mm, 92 parts, among them J1 24V IN, J10 TH1, J11 VFAN_SEL, J2 USB4105-GF-A, J3 FAN0, J4 FAN1, J5 FAN2, J6 TH0, J7 FAN3, J8 FAN4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

Commit message: Finished V1
Parts:
- removed C15: 22uF, Capacitor_SMD:C_0805_2012Metric
- removed U5: LM2940G-12V, Package_TO_SOT_SMD:SOT-223
- added D12: S1A, Diode_SMD:D_SMA, F.Cu at (127.3, 101.1)
- moved C14 49.6 mm to (186.5, 87.0), turned to -90 degrees
- moved R1 46.5 mm to (169.8, 87.6), turned to 180 degrees
- moved C16 46.0 mm to (189.8, 89.6)
- moved R5 44.1 mm to (189.8, 87.3)
- moved JP1 43.4 mm to (184.7, 99.8), turned to 90 degrees
- moved C4 40.2 mm to (190.6, 105.1), turned to 180 degrees
- moved C7 29.4 mm to (181.1, 104.6), turned to 90 degrees
- moved C18 29.2 mm to (157.6, 104.4), turned to 90 degrees
- moved Y1 27.8 mm to (185.7, 104.2)
- moved R2 25.8 mm to (190.6, 102.8), turned to 180 degrees
- moved C21 24.5 mm to (162.9, 104.4), turned to 90 degrees
- moved C8 23.9 mm to (177.2, 101.6), turned to 180 degrees
- moved C6 23.1 mm to (177.2, 99.2), turned to 180 degrees
- moved C20 21.1 mm to (160.3, 104.4), turned to 90 degrees
- moved F1 10.2 mm to (171.0, 96.4)
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Connections:
- net /USB+ renamed /D+
- net /USB- renamed /D-
- U4 pad 38: TH0 -> TH1
- U4 pad 39: TH1 -> TH0
Routing:
- net +3.3V: track 47.3 -> 155.8 mm, vias 5 -> 11
- net TH1: track 2.66 -> 99.6 mm, vias 0 -> 2
- net FAN5: track 2.60 -> 98.6 mm, vias 0 -> 2
- net TH0: track 2.66 -> 92.1 mm, vias 0 -> 2
- net FAN4: track 2.60 -> 90.7 mm, vias 0 -> 2
- net FAN3: track 2.60 -> 82.4 mm, vias 0 -> 2
- net FAN2: track 2.60 -> 73.5 mm, vias 0 -> 2
- net VFAN: track 0.00 -> 65.9 mm, vias 0 -> 1
- net FAN1: track 2.60 -> 63.4 mm, vias 0 -> 2
- net +5V: track 23.5 -> 75.7 mm, vias 1 -> 2
- net FAN0: track 2.60 -> 54.7 mm, vias 0 -> 2
- net SD0: track 2.52 -> 16.9 mm, vias 1 -> 2
- net CLK: track 2.23 -> 14.7 mm, vias 1 -> 2
- net Net-(C4-Pad2): track 0.00 -> 11.8 mm
- net Net-(C7-Pad1): track 0.00 -> 11.8 mm
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Other:
- board size 105 x 32 mm -> 105 x 30 mm
- board text added: "Better Klipper Expander V1"

Commit message: Vias, Widths, and Organization...
Parts:
- removed D12: S1A, Diode_SMD:D_SMA
- added F3: 4A, Fuse:Fuse_0805_2012Metric, F.Cu at (144.3, 100.2)
- J11: footprint Connector_PinSocket_2.54mm:PinSocket_2x02_P2.54mm_Vertical -> Connector_PinHeader_2.54mm:PinHeader_2x02_P2.54mm_Vertical
- moved C18 23.0 mm to (179.9, 98.8), turned to 180 degrees
- moved C21 21.1 mm to (183.5, 99.8), turned to 0 degrees
- moved C20 20.0 mm to (179.9, 100.8), turned to 180 degrees
- moved JP1 2.70 mm to (187.4, 99.7)
- moved L2 2.11 mm to (174.1, 98.8), turned to 0 degrees
- moved C8 1.10 mm to (176.1, 101.5)
- moved C6 0.72 mm to (176.8, 98.6), turned to 90 degrees
- moved G*** 0.66 mm to (93.3, 103.6)
- moved C9 0.64 mm to (173.4, 96.8), turned to 0 degrees
- moved Y1 0.50 mm to (185.2, 104.2)
- moved C4 0.49 mm to (190.1, 105.1)
- moved R2 0.49 mm to (190.1, 102.8)
- moved J11 0.37 mm to (116.3, 99.4)
- moved C14 0.36 mm to (186.7, 87.3)
- moved C7 0.30 mm to (180.8, 104.6)
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Connections:
- D10 pad 1: VFAN -> Net-(J9-Pad1)
- D10 pad 2: Net-(D10-Pad2) -> GND
- F1 pad 1: +5V -> Net-(C9-Pad1)
- F1 pad 2: Net-(C9-Pad1) -> +5V
- J11 pad 4: +5V -> Net-(J11-Pad4)
- J9 pad 1: Net-(D10-Pad2) -> Net-(J9-Pad1)
- J9 pad 2: VFAN -> GND
- Q6 pad 2: GND -> VFAN
- Q6 pad 3: Net-(D10-Pad2) -> Net-(J9-Pad1)
Routing:
- net +5V: track 75.7 -> 41.5 mm
- net Net-(J11-Pad4): track 0.00 -> 29.6 mm, vias 0 -> 1
- net Net-(J9-Pad1): track 0.00 -> 26.4 mm, vias 0 -> 1
- net Net-(D10-Pad2): track 21.7 -> 0.00 mm, vias 1 -> 0
- net +3.3V: track 155.8 -> 171.8 mm, vias 11 -> 14
- net GND: track 102.4 -> 92.6 mm, vias 26 -> 27
- net VFAN: track 65.9 -> 73.7 mm, vias 1 -> 2
- net Net-(L2-Pad2): track 5.17 -> 8.52 mm
- net Net-(U4-Pad21): track 10.3 -> 7.53 mm, vias 0 -> 2
- net Net-(C9-Pad1): track 6.70 -> 4.12 mm
- net VCC: track 76.4 -> 73.9 mm, vias 3 -> 2
- net FAN4: track 90.7 -> 89.3 mm
- net Net-(C7-Pad2): track 4.24 -> 5.58 mm
- net Net-(C4-Pad2): track 11.8 -> 13.0 mm
- net Net-(C7-Pad1): track 11.8 -> 11.3 mm, vias 0 -> 2
Other:
- board text added: "FAN0"
- board text added: "FAN1"
- board text added: "FAN2"
- board text added: "FAN3"
- board text added: "FAN4"
- board text added: "FAN5"

Commit message: Neopixelssssss....
Parts:
- removed R1: 5.1K, Resistor_SMD:R_0805_2012Metric
- added J12: Neopixel, Connector_PinHeader_2.54mm:PinHeader_1x03_P2.54mm_Vertical, F.Cu at (158.0, 104.2)
- added U5: TXS0101DBVR, TXS0101DBVR:SOT95P280X145-6N, F.Cu at (162.2, 104.3)
- R3, R4: value 27R -> 22R
- U1: value W25Q80DVSNIG_TR -> W25Q80DVSNIG
- U2: footprint Package_TO_SOT_SMD:SOT-23_Handsoldering -> Package_TO_SOT_SMD:SOT-23
- Y1: footprint Oscillator:Oscillator_SMD_SeikoEpson_SG8002CE-4Pin_3.2x2.5mm_HandSoldering -> Oscillator:Oscillator_SMD_SeikoEpson_SG8002CE-4Pin_3.2x2.5mm
Connections:
- net /D+ renamed D+
- net /D- renamed D-
- net Net-(C7-Pad1) renamed XIN
- net Net-(U4-Pad21) renamed XOUT
- F3 pad 1: Net-(J11-Pad4) -> Net-(F3-Pad1)
- J11 pad 3: VCC -> Net-(F3-Pad1)
- J11 pad 4: Net-(J11-Pad4) -> VCC
- J2 pad A5: Net-(J2-PadA5) -> unconnected-(J2-PadA5)
- J2 pad B5: Net-(J2-PadA5) -> unconnected-(J2-PadB5)
- U4 pad 36: unconnected-(U4-Pad36) -> GPIO24
Routing:
- net GPIO24: track 0.00 -> 30.9 mm, vias 0 -> 2
- net Net-(J11-Pad4): track 29.6 -> 0.00 mm, vias 1 -> 0
- net Net-(F3-Pad1): track 0.00 -> 29.6 mm, vias 0 -> 1
- net Net-(J2-PadA5): track 7.62 -> 0.00 mm
- net NEO_DATA: track 0.00 -> 6.59 mm
- net +5V: track 41.5 -> 47.8 mm
- net GND: track 92.6 -> 86.4 mm, vias 27 -> 28
- net FAN4: track 89.3 -> 84.5 mm
- net +3.3V: track 171.8 -> 176.0 mm
- net FAN1: track 63.1 -> 59.3 mm
- net FAN0: track 54.4 -> 51.2 mm
- net FAN2: track 73.6 -> 70.4 mm
- net FAN3: track 82.0 -> 79.9 mm
- net TH0: track 92.1 -> 94.1 mm
- net TH1: track 99.9 -> 101.8 mm
Other:
- board text added: "Neopixel"

Commit message: 3 fans per voltage selection now
Parts:
- added J13: VFAN_SEL2, Connector_PinHeader_2.54mm:PinHeader_2x02_P2.54mm_Vertical, F.Cu at (113.0, 99.0)
- J11: value VFAN_SEL -> VFAN_SEL1
- moved J11 17.6 mm to (133.9, 99.0)
- moved F3 1.41 mm to (145.7, 100.4)
Routing:
- net VFAN: track 73.7 -> 82.9 mm, vias 2 -> 3
- net Net-(J13-Pad3): track 29.6 -> 35.7 mm
- net VCC: track 73.9 -> 79.2 mm
- net FAN2: track 70.4 -> 67.6 mm
- net +5V: track 47.8 -> 46.3 mm
- net GND: track 86.4 -> 85.2 mm
- net XIN: track 11.5 -> 10.9 mm
