File: better-klipper-expander.kicad_pcb (KiCad board)
At the start: 4 copper layers, 105 x 30 mm, 93 parts, among them J1 24V IN, J10 TH1, J11 VFAN_SEL1, J12 Neopixel, J13 VFAN_SEL2, J2 USB4105-GF-A, J3 FAN0, J4 FAN1, J5 FAN2, J6 TH0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

Commit message: Minor updates
Connections:
- net NEO_DATA renamed Net-(J12-Pad2)
- C10 pad 1: Net-(C10-Pad1) -> +3.3V
- C11 pad 1: Net-(C10-Pad1) -> +3.3V
- C12 pad 1: Net-(C10-Pad1) -> +3.3V
- U4 pad 23: Net-(C10-Pad1) -> +3.3V
- U4 pad 45: Net-(C10-Pad1) -> +3.3V
- U4 pad 50: Net-(C10-Pad1) -> +3.3V
Routing:
- net +3.3V: track 175.6 -> 198.8 mm, vias 14 -> 18
- net Net-(C10-Pad1): track 23.0 -> 0.00 mm, vias 4 -> 0
- net VCC: track 79.2 -> 78.4 mm
- net SD2: track 5.95 -> 5.21 mm
- net SD1: track 5.55 -> 4.84 mm
- added copper zone on B.Cu, net GND
- added copper zone on In2.Cu, net GND

Commit message: change flash + fix major problem + minor cleanup
Parts:
- added C15: 0.1uF, Capacitor_SMD:C_0805_2012Metric, F.Cu at (184.6, 86.2)
- added G***: LOGO, Open Source Hardware:Open Source Hardware 5mm, F.Cu at (145.7, 103.4)
- C7, C8: footprint Capacitor_SMD:C_0805_2012Metric -> Capacitor_SMD:C_0603_1608Metric
- U1: value W25Q80DVSNIG -> W25Q16JVUXIQ; footprint FDS8896:SOIC127P600X175-8N -> W25Q16JVUXIQ:SON50P300X200X60-9N
- moved F3 0.80 mm to (145.7, 99.6)
- moved U1 0.68 mm to (181.1, 82.9), turned to 0 degrees
Connections:
- net GPIO24 renamed NEOPIXEL
- D10 pad 1: Net-(D10-Pad1) -> VFAN
- J9 pad 1: Net-(D10-Pad1) -> VFAN
- Q6 pad 3: Net-(D10-Pad1) -> VFAN
- U1 pad 8: VCC -> Net-(C15-Pad1)
Routing:
- net VFAN: track 82.9 -> 128.6 mm, vias 3 -> 4
- net VCC: track 78.4 -> 48.5 mm, vias 2 -> 0
- net Net-(D10-Pad1): track 26.4 -> 0.00 mm, vias 1 -> 0
- net SD0: track 16.9 -> 6.90 mm, vias 2 -> 0
- net CLK: track 14.7 -> 8.14 mm, vias 2 -> 0
- net Net-(C15-Pad1): track 0.00 -> 4.38 mm
- net SD1: track 4.84 -> 8.88 mm
- net CS: track 5.52 -> 9.50 mm
- net SD2: track 5.21 -> 7.94 mm
- net Net-(C13-Pad1): track 8.55 -> 6.66 mm
- net SD3: track 10.3 -> 8.78 mm, vias 2 -> 0
- net +3.3V: track 198.8 -> 200.2 mm
- net Net-(F3-Pad1): track 35.7 -> 34.8 mm
- net Net-(J12-Pad2): track 6.59 -> 5.73 mm
Other:
- board text added: "Boot"
- board text added: "JLCJLCJLC"
- board text added: "github.com/Fisheiyy/better-klipper-expander"
